File: CH554-USB-Devboard.sch (KiCad schematic (older format))
At the start: 20 parts, among them J1 Conn_01x10_Male, J2 Conn_01x10_Male, J3 USB_B_Micro, SW1 SW_Push, SW2 SW_Push, U1 CH552T, U2 CH552G, Y1 Crystal

Commit message: relinked libs
Parts:
- U1: symbol MCU_WCH:CH552T -> CH554-USB-Devboard-rescue:CH552T-MCU_WCH
- U2: symbol MCU_WCH:CH552G -> CH554-USB-Devboard-rescue:CH552G-MCU_WCH
Changed lines of the file:
@@
 EESchema Schematic File Version 4
-LIBS:CH552-USB-Devboard-cache
-EELAYER 26 0
+EELAYER 30 0
 EELAYER END
 $Descr A4 11693 8268
@@
 $EndComp
 $Comp
-L MCU_WCH:CH552T U1
+L CH554-USB-Devboard-rescue:CH552T-MCU_WCH U1
 U 1 1 5E91FA86
 P 3800 5200
@@
 $EndComp
 $Comp
-L MCU_WCH:CH552G U2
+L CH554-USB-Devboard-rescue:CH552G-MCU_WCH U2
 U 1 1 5E91FB0A
 P 8550 5500

Commit message: needs  VBUS to VCC control
Parts:
- removed C4: 100nF, Capacitor_SMD:C_0603_1608Metric_Pad1.05x0.95mm_HandSolder, symbol Device:C_Small
- removed J3: USB_B_Micro, digikey-footprints:USB_Micro_B_Female_10118193-0001LF, symbol Connector:USB_B_Micro
- removed U1: CH552T, Housings_SSOP:TSSOP-20_4.4x6.5mm_Pitch0.65mm, symbol CH554-USB-Devboard-rescue:CH552T-MCU_WCH
- removed U2: CH552G, Housings_SOIC:SOIC-16_3.9x9.9mm_Pitch1.27mm, symbol CH554-USB-Devboard-rescue:CH552G-MCU_WCH
- added C?: 100uF, Capacitor_SMD:C_0603_1608Metric_Pad1.05x0.95mm_HandSolder, symbol Device:C_Small
- added D?: D, symbol Device:D
- added J?: USB_C_Receptacle, symbol Connector:USB_C_Receptacle
- added JP? (x4): Jumper_NC_Small, symbol Device:Jumper_NC_Small
- added Q?: Q_PMOS_DSG, symbol Device:Q_PMOS_DSG
- added R? (x2): 10k, Resistor_SMD:R_0603_1608Metric_Pad1.05x0.95mm_HandSolder, symbol Device:R_Small
- added U?: CH554T, symbol MCU_WCH:CH554T
- added U?: CH554G, symbol MCU_WCH:CH554G
- added U?: AP22814, symbol Diodes_inc:AP22814
- C5, C6: value 100uF -> 15pF
Connections:
- net labels added: CC1, CC2, VBUS, enable
- wire segments 117 -> 167
Other:
- note added: "Optional External Crystal (HC49)\n"
- note added: "Reverse Protection Diode\n"
- note added: "used for downstream power issues \n"
- note added: "wrong at the moment as the body diode allows unwanted flow of current to VBUS"
- moved on the sheet: C5, C6, J1, J2, Y1

Commit message: schematic complete started to route
Parts:
- removed C?: 100uF, Capacitor_SMD:C_0603_1608Metric_Pad1.05x0.95mm_HandSolder, symbol Device:C_Small
- removed JP? (x2): Jumper_NC_Small, symbol Device:Jumper_NC_Small
- removed Q?: Q_PMOS_DSG, symbol Device:Q_PMOS_DSG
- removed R? (x2): 10k, Resistor_SMD:R_0603_1608Metric_Pad1.05x0.95mm_HandSolder, symbol Device:R_Small
- removed U?: AP22814, symbol Diodes_inc:AP22814
- added C4, C7: 100nF, Capacitor_SMD:C_0603_1608Metric_Pad1.05x0.95mm_HandSolder, symbol Device:C_Small
- added JP1: Jumper_3_Bridged12, Jumper:SolderJumper-3_P1.3mm_Bridged12_RoundedPad1.0x1.5mm_NumberLabels, symbol Jumper:Jumper_3_Bridged12
- added JP2, JP3: Jumper_NC_Small, Jumper:SolderJumper-2_P1.3mm_Bridged_RoundedPad1.0x1.5mm, symbol Device:Jumper_NC_Small
- added Q1, Q2: CPH6337, TO_SOT_Packages_SMD:SOT-23-6, symbol OnSemi:CPH6337
- added R1, R2: 10k, Resistor_SMD:R_0603_1608Metric_Pad1.05x0.95mm_HandSolder, symbol Device:R_Small
- added U2: MIC5504-3.3YM5, Package_TO_SOT_SMD:SOT-23-5, symbol Regulator_Linear:MIC5504-3.3YM5
- D4: renamed from D?; value D -> SMBJ58A+; footprint (none) -> Diode_SMD:D_1812_4532Metric
- JP4, JP5: renamed from JP?; footprint (none) -> Jumper:SolderJumper-2_P1.3mm_Bridged_RoundedPad1.0x1.5mm
- U1: renamed from U?; footprint (none) -> Housings_SSOP:TSSOP-20_4.4x6.5mm_Pitch0.65mm
- U3: renamed from U?; footprint (none) -> Housings_SOIC:SOIC-16_3.9x9.9mm_Pitch1.27mm
- gave numbers to parts that had none: 1
Connections:
- net labels added: VSYS
- net labels removed: enable
- wire segments 167 -> 174
Other:
- note added: "Device mode VBUS ->VCC P3.4 = 0/z P1.1 = 1/z (default)\nHost mode VCC ->VBUS P3.4 = 1 P1.1 = 0 \nPower Freeflow VCC <-> VBUS P3.4 = 0/z P1.1 = 0"
- note removed: "used for downstream power issues \n"
- note removed: "wrong at the moment as the body diode allows unwanted flow of current to VBUS"

Commit message: more routing
Changed lines of the file:
@@
 Wire Wire Line
 	6700 6100 7300 6100
+Text Label 6700 6100 0    50   ~ 0
+P3.0
 Text Label 6700 5950 0    50   ~ 0
-P3.0
-Text Label 6700 6100 0    50   ~ 0
 P3.1
 Text Label 6700 5050 0    50   ~ 0
@@
 	1    0    0    -1
 $EndComp
+Text Label 9600 2150 2    50   ~ 0
+P3.0
 Text Label 9600 1800 2    50   ~ 0
-P3.0
-Text Label 9600 2150 2    50   ~ 0
 P3.1
 Text Notes 9800 1850 2    50   ~ 0
@@
 Wire Wire Line
 	4050 1050 4050 850
-$Comp
-L power:VCC #PWR0114
-U 1 1 5E94BA61
-P 4050 850
-F 0 "#PWR0114" H 4050 700 50  0001 C CNN
-F 1 "VCC" H 4067 1023 50  0000 C CNN
-F 2 "" H 4050 850 50  0001 C CNN
-F 3 "" H 4050 850 50  0001 C CNN
-	1    4050 850
-	1    0    0    -1
-$EndComp
 $Comp
 L Switch:SW_Push SW2
@@
 	0    -1   1    0
 $EndComp
+Text Label 4050 850  0    50   ~ 0
+VSYS
 $EndSCHEMATC
